File: old/m2/m2/m2.kicad_pcb (KiCad board)
At the start: 4 copper layers, 101.2 x 76.2 mm, 21 parts, among them CN1 PJ-332A-6A, CN2 PJ-332A-6A, CN3 Pogo Pin Receptor Right, CN4 Battery connector JST-PH, SW1 TS24CA 250GF 013, SW2 TS24CA 250GF 013, U1 SLSS49E-3, U2 SLSS49E-3, U3 SLSS49E-3, U4 SLSS49E-3, U5 SLSS49E-3, U6 H11L1S(TA), U7 Pogo Pin Left, U8 AP2112K-3.3

Commit message: added version 1.0 of kicad file for kh-24
some eva inspired posters too, have fun
Routing:
- net DP_PRE: track 0.00 -> 7.54 mm
Changed lines of the file:
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@@
+	)
+	(segment
+		(start 74.536 36.97)
+		(end 75.95 35.556)
+		(width 0.2)
+		(layer "B.Cu")
+		(net 79)
+	)
+	(segment
+		(start 70.59 36.97)
+		(end 74.536 36.97)
+		(width 0.2)
+		(layer "B.Cu")
+		(net 79)
+	)
+	(segment
+		(start 75.95 35.556)
+		(end 75.95 33.966)
+		(width 0.2)
+		(layer "B.Cu")
+		(net 79)
 	)
 	(segment
