File: kh-24 hall/kh-24/kh-24.kicad_sch (KiCad schematic)
At the start: 59 parts, among them CN3 Pogo Pin Receptor Right, J1 Conn_01x06, Q1 AO3400A, Q2 AO3400A, U1 SLSS49E-3, U10 SLSS49E-3, U11 H3V3U10B, U12 SLSS49E-3, U13 SLSS49E-3, U14 SLSS49E-3, U15 SLSS49E-3, U16 SLSS49E-3, U17 SLSS49E-3, U18 CD4051BM96, U19 SLSS49E-3, U2 ATtiny1616-M, U20 SLSS49E-3, U21 SLSS49E-3, U24 SLSS49E-3, U25 SLSS49E-3, U26 CD4051BM96, U27 SLSS49E-3, U28 SLSS49E-3, U29 SLSS49E-3, U3 CD4051BM96, U30 SLSS49E-3, U31 SLSS49E-3, U32 SLSS49E-3, U33 SLSS49E-3, U34 CD4051BM96, U35 SLSS49E-3, U4 SLSS49E-3, U5 H3V3U10B, U6 SLSS49E-3, U7 Pogo Pin Left, U8 AP2112K-3.3, U9 SLSS49E-3

Commit message: km-5 mostly finished
Connections:
- no-connect marks 9 -> 12
Changed lines of the file:
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@@
+	)
+	(no_connect
+		(at 60.96 111.76)
 	)
 	(no_connect
@@
 	)
 	(no_connect
+		(at 60.96 109.22)
+	)
+	(no_connect
 		(at 340.36 1.27)
 	)
 	(no_connect
+		(at 60.96 114.3)
+	)
+	(no_connect

Commit message: work
Parts:
- removed Q1, Q2: AO3400A, Package_TO_SOT_SMD:SOT-23, symbol Transistor_FET:AO3400A
- removed R5, R6, R7, R8: 10K, Resistor_SMD:R_0402_1005Metric, symbol Device:R
- added C8: 1u, Capacitor_SMD:C_0402_1005Metric, symbol Device:C
- added Q1, Q3: AO3401A, Package_TO_SOT_SMD:SOT-23, symbol Transistor_FET:AO3401A
- added R9: 10K, Resistor_SMD:R_0402_1005Metric, symbol Device:R
- added U22: LM66200DRLR, easyeda2kicad:SOT-583-8_L2.1-W1.2-P0.50-LS1.6-BL, symbol easyeda2kicad:LM66200DRLR
Connections:
- net GND: now also U22.1 (GND), U22.4 (~{ON}), U22.5 (GND)
- net PWR: now also C8.1, Q1.1 (G), Q3.1 (G), R9.2
- net VBUS: now also U22.2 (VOUT), U22.7 (VOUT)
- net VBUS0: now also Q1.3 (D), U22.6 (VIN2)
- net VBUS1: now also Q3.3 (D), U22.3 (VIN1)
- new net: C8.2, Q1.2 (S), Q3.2 (S), R9.1
- no-connect marks 12 -> 14

Commit message: many
Parts:
- added KEY1, KEY10, KEY11, KEY12, KEY13, KEY14, KEY15, KEY16, KEY17, KEY18, KEY19, KEY2, KEY20, KEY21, KEY22, KEY23, KEY24, KEY3, KEY4, KEY5, KEY6, KEY7, KEY8, KEY9: 28115181DM, copper:hall_key_footprint, symbol easyeda2kicad:28115181DM

Commit message: production 1
Parts:
- added R5, R6, R7, R8: 10K, Resistor_SMD:R_0402_1005Metric_Pad0.72x0.64mm_HandSolder, symbol Device:R
Connections:
- net A0: now also R5.1
- net A1: now also R6.1
- net A2: now also R7.1
- net A3: now also R8.1
- net GND: now also R5.2, R6.2, R7.2, R8.2
