File: km-05 mod/km-05/km-05.kicad_pcb (KiCad board)
At the start: 4 copper layers, 50.8 x 153.7 mm, 64 parts, among them CN1 YTC1P-6030-01, CN10 YTC1P-6030-01, CN11 YTC1P-6030-01, CN12 YTC1P-6030-01, CN13 YTC1P-6030-01, CN14 YTC1P-6030-01, CN2 YTC1P-6030-01, CN3 Pogo Pin Receptor Right, CN4 YTC1P-6030-01, CN5 YTC1P-6030-01, CN6 YTC1P-6030-01, CN7 YTC1P-6030-01, CN8 YTC1P-6030-01, CN9 YTC1P-6030-01, J1 Conn_01x06, Q1 AO3400A, Q2 AO3400A, U1 H3V3U10B, U10 H3V3U10B, U11 H3V3U10B, U12 H3V3U10B, U13 H3V3U10B, U14 H3V3U10B, U15 H3V3U10B, U16 H3V3U10B, U17 H3V3U10B, U18 H3V3U10B, U2 ATtiny1616-M, U3 H3V3U10B, U4 H3V3U10B, U5 H3V3U10B, U6 H3V3U10B, U7 Pogo Pin Left, U8 AP2112K-3.3, U9 H3V3U10B

Commit message: km-5 mostly finished
Parts:
- removed CN13: YTC1P-6030-01, easyeda2kicad:SMD-1_BD2.0-H10.0
- added R21: 10K, Resistor_SMD:R_0402_1005Metric, F.Cu at (80.3, 34.6)
- added R22: 10K, Resistor_SMD:R_0402_1005Metric, F.Cu at (81.9, 48.7)
- added R23: 10K, Resistor_SMD:R_0402_1005Metric, F.Cu at (83.7, 63.6)
- added R24: 10K, Resistor_SMD:R_0402_1005Metric, F.Cu at (79.5, 74.1)
- added R25: 10K, Resistor_SMD:R_0402_1005Metric, F.Cu at (95.1, 41.0)
- added R26: 10K, Resistor_SMD:R_0402_1005Metric, F.Cu at (85.0, 49.1)
- added R27: 10K, Resistor_SMD:R_0402_1005Metric, F.Cu at (83.4, 55.0)
- added R28: 10K, Resistor_SMD:R_0402_1005Metric, F.Cu at (90.0, 74.8)
- added U19: SK6812MINI-HS, easyeda2kicad:LED-SMD_4P-L3.5-W3.5-BR_SK6812MINI-HS, F.Cu at (79.3, 48.2)
- added U20: SK6812MINI-HS, easyeda2kicad:LED-SMD_4P-L3.5-W3.5-BR_SK6812MINI-HS, F.Cu at (79.3, 70.0)
- added U21: SK6812MINI-HS, easyeda2kicad:LED-SMD_4P-L3.5-W3.5-BR_SK6812MINI-HS, F.Cu at (79.3, 91.8)
- added U22: SK6812MINI-HS, easyeda2kicad:LED-SMD_4P-L3.5-W3.5-BR_SK6812MINI-HS, F.Cu at (90.7, 91.7)
- added U23: SK6812MINI-HS, easyeda2kicad:LED-SMD_4P-L3.5-W3.5-BR_SK6812MINI-HS, F.Cu at (90.7, 69.9)
- added U24: SK6812MINI-HS, easyeda2kicad:LED-SMD_4P-L3.5-W3.5-BR_SK6812MINI-HS, F.Cu at (90.7, 48.2)
- added U25: SK6812MINI-HS, easyeda2kicad:LED-SMD_4P-L3.5-W3.5-BR_SK6812MINI-HS, F.Cu at (90.7, 26.4)
- U1: value H3V3U10B -> SK6812MINI-HS; footprint easyeda2kicad:DFN1006-2L-BI -> easyeda2kicad:LED-SMD_4P-L3.5-W3.5-BR_SK6812MINI-HS
- moved U11 166.7 mm to (69.2, 50.4), turned to 90 degrees
- moved U5 162.6 mm to (69.2, 55.0), turned to -90 degrees
- moved U18 162.2 mm to (64.0, 43.6), turned to 90 degrees
- moved R12 157.8 mm to (94.8, 46.2), turned to 180 degrees
- moved R11 157.6 mm to (94.8, 45.2), turned to 180 degrees
- moved R10 157.5 mm to (94.8, 44.2), turned to 180 degrees
- moved R19 157.4 mm to (98.9, 42.9), turned to 90 degrees
- moved R18 156.1 mm to (99.9, 42.9), turned to 90 degrees
- moved R9 155.9 mm to (96.3, 42.9), turned to 90 degrees
- moved R16 155.8 mm to (98.6, 51.6), turned to -90 degrees
- moved R15 154.7 mm to (99.6, 51.6), turned to -90 degrees
- moved R17 154.2 mm to (101.2, 44.7)
- moved R14 151.8 mm to (100.6, 51.6), turned to -90 degrees
- moved R13 150.5 mm to (101.6, 51.6), turned to -90 degrees
- moved C7 149.3 mm to (70.6, 73.4)
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Connections:
- R10 pad 2: Net-(CN2-Pad1) -> Net-(CN8-Pad1)
- R11 pad 2: Net-(CN4-Pad1) -> Net-(CN2-Pad1)
- R12 pad 2: Net-(CN5-Pad1) -> Net-(CN7-Pad1)
- R13 pad 2: Net-(CN6-Pad1) -> Net-(CN11-Pad1)
- R14 pad 2: Net-(CN7-Pad1) -> Net-(CN10-Pad1)
- R15 pad 2: Net-(CN8-Pad1) -> Net-(CN5-Pad1)
- R16 pad 2: Net-(CN9-Pad1) -> Net-(CN6-Pad1)
- R17 pad 2: Net-(CN10-Pad1) -> Net-(CN14-Pad1)
- R18 pad 2: Net-(CN11-Pad1) -> Net-(CN12-Pad1)
- R19 pad 2: Net-(CN12-Pad1) -> Net-(CN9-Pad1)
- R20 pad 2: Net-(CN14-Pad1) -> Net-(CN4-Pad1)
- U10 pad 2: A4 -> Net-(CN14-Pad1)
- U12 pad 2: A3 -> Net-(CN5-Pad1)
- U13 pad 2: A2 -> Net-(CN4-Pad1)
- U14 pad 2: A1 -> Net-(CN2-Pad1)
- U15 pad 2: A0 -> Net-(CN1-Pad1)
- U16 pad 2: A16 -> Net-(CN12-Pad1)
- U17 pad 2: A15 -> Net-(CN11-Pad1)
- U18 pad 2: A14 -> Net-(CN10-Pad1)
- U3 pad 2: D10 -> Net-(CN9-Pad1)
- U4 pad 2: D11 -> Net-(CN8-Pad1)
- U6 pad 2: D12 -> Net-(CN7-Pad1)
- U9 pad 2: D13 -> Net-(CN6-Pad1)
Routing:
- net PWR: track 0.00 -> 72.4 mm, vias 0 -> 2
- net Net-(CN5-Pad1): track 0.00 -> 56.9 mm, vias 0 -> 2
- net Net-(CN10-Pad1): track 0.00 -> 52.2 mm, vias 0 -> 2
- net Net-(CN6-Pad1): track 0.00 -> 50.1 mm, vias 0 -> 5
- net Net-(CN7-Pad1): track 0.00 -> 46.9 mm, vias 0 -> 3
- net Net-(CN11-Pad1): track 0.00 -> 42.0 mm, vias 0 -> 2
- net Net-(CN4-Pad1): track 0.00 -> 40.1 mm, vias 0 -> 3
- net GND: track 0.00 -> 36.7 mm, vias 1 -> 50
- net NEO: track 0.00 -> 35.6 mm, vias 0 -> 4
- net Net-(CN2-Pad1): track 0.00 -> 35.1 mm, vias 0 -> 3
- net Net-(CN1-Pad1): track 0.00 -> 33.4 mm, vias 0 -> 2
- net Net-(U24-DOUT): track 0.00 -> 30.5 mm, vias 0 -> 3
- net SDA0: track 48.9 -> 77.3 mm, vias 0 -> 2
- net Net-(CN14-Pad1): track 0.00 -> 28.2 mm, vias 0 -> 2
- net Net-(CN12-Pad1): track 0.00 -> 27.3 mm
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- added copper zone on F.Cu, net cn1-pad2
- added copper zone on F.Cu, net cn12-Pad2
- added copper zone on F.Cu, net cn14-pad2
- added copper zone on F.Cu, net cn2-pad2
- added copper zone on F.Cu, net cn4-pad2
- added copper zone on F.Cu, net cn5-pad2
- added copper zone on F.Cu, net cn6-pad2
- added copper zone on F.Cu, net cn7-pad2
- added copper zone on F.Cu, net cn8-pad2
- added copper zone on F.Cu, net cn9-pad2
Other:
- board size 50.8 x 153.7 mm -> 150.8 x 76.2 mm

Commit message: work
Parts:
- removed the H1 at (185.0, 40.0)
- removed the H1 at (185.0, 27.4)
- removed the H2 at (185.0, 78.0)
- removed the H2 at (185.0, 90.8)
- removed Q1, Q2: AO3400A, Package_TO_SOT_SMD:SOT-23
- removed R5, R6, R7, R8: 10K, Resistor_SMD:R_0402_1005Metric
- added C8: 1u, Capacitor_SMD:C_0402_1005Metric, F.Cu at (67.2, 63.4)
- added Q3: AO3401A, Package_TO_SOT_SMD:SOT-23, F.Cu at (66.8, 65.9)
- added Q4: AO3401A, Package_TO_SOT_SMD:SOT-23, F.Cu at (66.7, 70.3)
- added R29: 10K, Resistor_SMD:R_0402_1005Metric, F.Cu at (67.2, 62.4)
- added U26: LM66200DRLR, easyeda2kicad:SOT-583-8_L2.1-W1.2-P0.50-LS1.6-BL, F.Cu at (66.2, 73.4)
Routing:
- net cn14-pad2: track 12.0 -> 0.00 mm, vias 1 -> 0
- net cn12-Pad2: track 11.0 -> 0.00 mm, vias 1 -> 0
- net VBUS: track 17.2 -> 9.57 mm
- net Net-(Q3-S): track 0.00 -> 7.38 mm
- net VBUS0: track 16.8 -> 23.9 mm, vias 0 -> 2
- net cn1-pad2: track 6.86 -> 0.00 mm, vias 1 -> 0
- net cn9-pad2: track 5.80 -> 0.00 mm, vias 1 -> 0
- net cn2-pad2: track 5.75 -> 0.00 mm, vias 1 -> 0
- net PWR: track 72.4 -> 76.9 mm
- net cn5-pad2: track 4.43 -> 0.00 mm, vias 1 -> 0
- net cn4-pad2: track 4.37 -> 0.00 mm, vias 1 -> 0
- net cn6-pad2: track 3.94 -> 0.00 mm, vias 1 -> 0
- net cn8-pad2: track 3.80 -> 0.00 mm, vias 1 -> 0
- net cn7-pad2: track 3.58 -> 0.00 mm, vias 1 -> 0
- net GND: track 36.7 -> 39.6 mm
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- removed copper zone on F.Cu, net cn1-pad2
- removed copper zone on F.Cu, net cn12-Pad2
- removed copper zone on F.Cu, net cn14-pad2
- removed copper zone on F.Cu, net cn2-pad2
- removed copper zone on F.Cu, net cn4-pad2
- removed copper zone on F.Cu, net cn5-pad2
- removed copper zone on F.Cu, net cn6-pad2
- removed copper zone on F.Cu, net cn7-pad2
- removed copper zone on F.Cu, net cn8-pad2
- removed copper zone on F.Cu, net cn9-pad2
Other:
- board size 150.8 x 76.2 mm -> 50.3 x 71.2 mm

Commit message: core mainboard
Routing:
- net GND: vias 50 -> 59

Commit message: many
Other:
- board text added: "0.1"
- board text added: "2/2026"
- board text added: "3.3V"
- board text added: "CC-BY-NC-SA 4.0"
- board text added: "DESIGN"
- board text added: "GITHUB.COM/TORBERS"
- board text added: "GND"
- board text added: "MODS"
- board text added: "OPEN SOURCE"
- board text added: "SCL"
- board text added: "SDA"
- board text added: "SHEPHERD MIX MODULE"
- board text added: "SOURCE FILES"
- board text added: "TEST TYPE"
- board text added: "TORBERS"
- board text added: "TXD"
- board text added: "UPDI"
- board text added: "VBUS"

Commit message: prod
Parts:
- C6, C7: value 1u -> 10u
- R10, R11, R12, R13, R14, R15, R16, R17, R18, R19, R20, R9: value 1K -> 0R
- moved R17 0.22 mm to (101.2, 44.5)
Connections:
- U2 pad 1: A15 -> SCL0
- U2 pad 10: NEO -> A16
- U2 pad 13: SDA0 -> A15
- U2 pad 14: SCL0 -> A14
- U2 pad 2: A16 -> NEO
- U2 pad 20: A14 -> SDA0
Routing:
- net A16: track 1.75 -> 15.2 mm, vias 0 -> 2
- net A15: track 2.05 -> 11.3 mm, vias 0 -> 2
- net A14: track 1.61 -> 9.86 mm, vias 0 -> 2
- net TXD: track 14.1 -> 21.9 mm
- net Net-(CN10-Pad1): track 52.2 -> 45.1 mm
- net SDA0: track 77.3 -> 71.8 mm, vias 2 -> 1
- net SCL0: track 73.3 -> 69.8 mm, vias 2 -> 0
- net NEO: track 35.6 -> 33.3 mm, vias 4 -> 6
- net Net-(CN14-Pad1): track 28.2 -> 30.0 mm
- net GND: track 39.6 -> 37.9 mm, vias 59 -> 61
- net Net-(CN9-Pad1): track 21.9 -> 23.2 mm
