File: km-05 mod/km-05/km-05.kicad_pcb (KiCad board)
At the start: 4 copper layers, 50.3 x 71.2 mm, 73 parts, among them CN1 YTC1P-6030-01, CN10 YTC1P-6030-01, CN11 YTC1P-6030-01, CN12 YTC1P-6030-01, CN14 YTC1P-6030-01, CN2 YTC1P-6030-01, CN3 Pogo Pin Receptor Right, CN4 YTC1P-6030-01, CN5 YTC1P-6030-01, CN6 YTC1P-6030-01, CN7 YTC1P-6030-01, CN8 YTC1P-6030-01, CN9 YTC1P-6030-01, J1 Conn_01x06, Q3 AO3401A, Q4 AO3401A, U1 SK6812MINI-HS, U10 H3V3U10B, U11 H3V3U10B, U12 H3V3U10B, U13 H3V3U10B, U14 H3V3U10B, U15 H3V3U10B, U16 H3V3U10B, U17 H3V3U10B, U18 H3V3U10B, U19 SK6812MINI-HS, U2 ATtiny1616-M, U20 SK6812MINI-HS, U21 SK6812MINI-HS, U22 SK6812MINI-HS, U23 SK6812MINI-HS, U24 SK6812MINI-HS, U25 SK6812MINI-HS, U26 LM66200DRLR, U3 H3V3U10B, U4 H3V3U10B, U5 H3V3U10B, U6 H3V3U10B, U7 Pogo Pin Left, U8 AP2112K-3.3, U9 H3V3U10B

Commit message: production 1
Parts:
- added G***: LOGO, LOGO, F.Cu at (102.9, 68.9)
