File: km-05 mod/km-05/km-05.kicad_sch (KiCad schematic)
At the start: 60 parts, among them CN1 YTC1P-6030-01, CN10 YTC1P-6030-01, CN11 YTC1P-6030-01, CN12 YTC1P-6030-01, CN13 YTC1P-6030-01, CN14 YTC1P-6030-01, CN2 YTC1P-6030-01, CN3 Pogo Pin Receptor Right, CN4 YTC1P-6030-01, CN5 YTC1P-6030-01, CN6 YTC1P-6030-01, CN7 YTC1P-6030-01, CN8 YTC1P-6030-01, CN9 YTC1P-6030-01, J1 Conn_01x06, Q1 AO3400A, Q2 AO3400A, U1 H3V3U10B, U10 H3V3U10B, U11 H3V3U10B, U12 H3V3U10B, U13 H3V3U10B, U14 H3V3U10B, U15 H3V3U10B, U16 H3V3U10B, U17 H3V3U10B, U18 H3V3U10B, U2 ATtiny1616-M, U3 H3V3U10B, U4 H3V3U10B, U5 H3V3U10B, U6 H3V3U10B, U7 Pogo Pin Left, U8 AP2112K-3.3, U9 H3V3U10B

Commit message: km-5 mostly finished
Parts:
- removed CN13: YTC1P-6030-01, easyeda2kicad:SMD-1_BD2.0-H10.0, symbol easyeda2kicad:YTC1P-6030-01
- removed U1: H3V3U10B, easyeda2kicad:DFN1006-2L-BI, symbol easyeda2kicad:H3V3U10B
- added R21, R22, R23, R24, R25, R26, R27, R28: 10K, Resistor_SMD:R_0402_1005Metric, symbol Device:R
- added U1, U19, U20, U21, U22, U23, U24, U25: SK6812MINI-HS, easyeda2kicad:LED-SMD_4P-L3.5-W3.5-BR_SK6812MINI-HS, symbol easyeda2kicad:SK6812MINI-HS
Connections:
- net +3.3V: now also U1.3 (VDD), U19.3 (VDD), U20.3 (VDD), U21.3 (VDD), U22.3 (VDD), U23.3 (VDD), U24.3 (VDD), U25.3 (VDD)
- net A0: no longer U15.2
- net A1: no longer U14.2
- net A14: no longer U18.2
- net A15: no longer U17.2
- net A16: no longer U16.2
- net A2: no longer U13.2
- net A3: no longer U12.2
- net A4: no longer U10.2
- net D10: no longer U3.2
- net D11: no longer U4.2
- net D12: no longer U6.2
- net D13: no longer U9.2
- net GND: now also U1.1 (GND), U19.1 (GND), U20.1 (GND), U21.1 (GND), U22.1 (GND), U23.1 (GND), U24.1 (GND), U25.1 (GND)
- net NEO: now also U1.2 (DIN)
- net at CN1.1, R9.2: now also U15.2, R21.2, R22.1
- net at CN7.1: now also R12.2, U6.2, R27.2, R28.1; no longer R14.2
- net at R18.2: now also CN12.1, U16.2, R21.1; no longer CN11.1
- net at CN5.1: now also R15.2, U12.2, R24.2; no longer R12.2
- net at CN8.1: now also R10.2, U4.2, R26.2, R27.1; no longer R15.2
- net at CN6.1: now also R16.2, U9.2, R28.2; no longer R13.2
- net at R20.2: now also CN4.1, U13.2, R23.2, R24.1; no longer CN14.1
- net at R19.2: now also CN9.1, U3.2, R25.2, R26.1; no longer CN12.1
- net at R11.2: now also CN2.1, U14.2, R22.2, R23.1; no longer CN4.1
- net at CN10.1: now also R14.2, U18.2; no longer R17.2
- new net: U24.4 (DOUT), U25.2 (DIN)
- new net: U23.4 (DOUT), U24.2 (DIN)
- new net: CN14.1, R17.2, R25.1, U10.2
- new net: CN11.1, R13.2, U17.2
- new net: U1.4 (DOUT), U19.2 (DIN)
- new net: U22.4 (DOUT), U23.2 (DIN)
- new net: U21.4 (DOUT), U22.2 (DIN)
- new net: U19.4 (DOUT), U20.2 (DIN)
- new net: U20.4 (DOUT), U21.2 (DIN)
- no-connect marks 0 -> 1
Other:
- note added: "NeoPixels"
- note removed: "Neopixel pin"
- note removed: "Reciever pins 2 cont."
- moved on the sheet: CN1, CN10, CN11, CN12, CN14, CN2, CN4, CN5, CN6, CN7, CN8, CN9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

Commit message: work
Parts:
- removed Q1, Q2: AO3400A, Package_TO_SOT_SMD:SOT-23, symbol Transistor_FET:AO3400A
- removed R5, R6, R7, R8: 10K, Resistor_SMD:R_0402_1005Metric, symbol Device:R
- added C8: 1u, Capacitor_SMD:C_0402_1005Metric, symbol Device:C
- added Q3, Q4: AO3401A, Package_TO_SOT_SMD:SOT-23, symbol Transistor_FET:AO3401A
- added R29: 10K, Resistor_SMD:R_0402_1005Metric, symbol Device:R
- added U26: LM66200DRLR, easyeda2kicad:SOT-583-8_L2.1-W1.2-P0.50-LS1.6-BL, symbol easyeda2kicad:LM66200DRLR
Connections:
- net GND: now also U26.1 (GND), U26.4 (~{ON}), U26.5 (GND)
- net PWR: now also C8.1, Q3.1 (G), Q4.1 (G), R29.2
- net VBUS: now also U26.2 (VOUT), U26.7 (VOUT)
- net VBUS0: now also Q3.3 (D), U26.6 (VIN2)
- net VBUS1: now also Q4.3 (D), U26.3 (VIN1)
- new net: C8.2, Q3.2 (S), Q4.2 (S), R29.1
- no-connect marks 1 -> 2

Commit message: core mainboard
Parts:
- R21, R22, R23, R24, R25, R26, R27, R28: now not fitted
Changed lines of the file:
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@@
 		(in_bom yes)
 		(on_board yes)
-		(dnp no)
+		(dnp yes)
 		(property "Reference" "R28"
 			(at 246.126 127.254 90)
@@
 		(in_bom yes)
 		(on_board yes)
-		(dnp no)
+		(dnp yes)
 		(property "Reference" "R21"
 			(at 246.126 43.434 90)
@@
 		(in_bom yes)
 		(on_board yes)
-		(dnp no)
+		(dnp yes)
 		(property "Reference" "R24"
 			(at 246.126 73.914 90)
@@
 		(in_bom yes)
 		(on_board yes)
-		(dnp no)
+		(dnp yes)
 		(property "Reference" "R26"
 			(at 246.126 106.934 90)
@@
 		(in_bom yes)
 		(on_board yes)
-		(dnp no)
+		(dnp yes)
 		(property "Reference" "R23"
 			(at 246.126 63.754 90)
@@
 		(in_bom yes)
 		(on_board yes)
-		(dnp no)
+		(dnp yes)
 		(property "Reference" "R22"
 			(at 246.126 53.594 90)
@@
 		(in_bom yes)
 		(on_board yes)
-		(dnp no)
+		(dnp yes)
 		(property "Reference" "R27"
 			(at 246.126 117.094 90)
@@
 		(in_bom yes)
 		(on_board yes)
-		(dnp no)
+		(dnp yes)
 		(property "Reference" "R25"
 			(at 246.126 96.774 90)

Commit message: prod
Parts:
- C6, C7: value 1u -> 10u
- R10, R11, R12, R13, R14, R15, R16, R17, R18, R19, R20, R9: value 1K -> 0R
Connections:
- net A14: now also U2.14 (PB0); no longer U2.20 (PA1)
- net A15: now also U2.13 (PB1); no longer U2.1 (PA2)
- net A16: now also U2.10 (PB4); no longer U2.2 (PA3)
- net NEO: now also U2.2 (PA3); no longer U2.10 (PB4)
- net SCL0: now also U2.1 (PA2); no longer U2.14 (PB0)
- net SDA0: now also U2.20 (PA1); no longer U2.13 (PB1)
